Commit message: Add sensors and improvements

File: nanosaur_gazebo/urdf/nanosaur.urdf.xacro (robot description, xacro)
@@ -5,6 +5,10 @@
     <!-- differential drive -->
     <xacro:include filename="$(find nanosaur_gazebo)/urdf/diff_drive.gazebo.xacro" />
+    <!-- Sensors -->
+    <xacro:include filename="$(find nanosaur_gazebo)/urdf/sensors/camera.gazebo.xacro" />
+    <xacro:include filename="$(find nanosaur_gazebo)/urdf/sensors/wide.gazebo.xacro" />
     <!-- camera definitions -->
     <xacro:arg name="cover_type" default="realsense" /> <!--options: pi, fisheye, realsense, zedmini -->
+    <xacro:property name="cover_type_name" value="$(arg cover_type)" />
     <!-- nanosaur robot
          "diff_drive_emulation" parameter enable simulation mode.
@@ -19,3 +23,18 @@
                        wheel_radius="0.0150"
                        wheel_separation="0.4" />
+    <!-- Nanosaur sensors -->
+    <xacro:if value="${cover_type_name == 'pi'}">
+        <xacro:normal_camera parent_name="camera_board" sensor_name="rgb_camera_nanosaur">
+            <origin xyz="0 0 0" rpy="0 ${M_PI/2} 0" />
+        </xacro:normal_camera>
+    </xacro:if>
+    <xacro:if value="${cover_type_name == 'fisheye'}">
+        <xacro:wide_angle_camera parent_name="camera_board" sensor_name="rgb_camera_nanosaur">
+            <origin xyz="0 0 0" rpy="0 0 0" />
+        </xacro:wide_angle_camera>
+    </xacro:if>
+    <xacro:if value="${cover_type_name == 'realsense'}">
+    </xacro:if>
+    <xacro:if value="${cover_type_name == 'zedmini'}">
+    </xacro:if>
 </robot>

Commit message: Fix camera pi

File: nanosaur_gazebo/urdf/nanosaur.urdf.xacro (robot description, xacro)
@@ -27,10 +27,10 @@
     <!-- Nanosaur sensors -->
     <xacro:if value="${cover_type_name == 'pi'}">
-        <xacro:normal_camera parent_name="camera_board" sensor_name="rgb_camera_nanosaur">
+        <xacro:normal_camera parent_name="camera_board" sensor_name="camera" robot_name="nanosaur">
             <origin xyz="0 0 0" rpy="0 ${M_PI/2} 0" />
         </xacro:normal_camera>
     </xacro:if>
     <xacro:if value="${cover_type_name == 'fisheye'}">
-        <xacro:wide_angle_camera parent_name="camera_board" sensor_name="rgb_camera_nanosaur">
+        <xacro:wide_angle_camera parent_name="camera_board" sensor_name="camera" robot_name="nanosaur">
             <origin xyz="0 0 0" rpy="0 0 0" />
         </xacro:wide_angle_camera>

File: nanosaur_gazebo/urdf/sensors/camera.gazebo.xacro (robot description, xacro)
@@ -6,7 +6,7 @@
     <xacro:property name="camera_box_y" value="0.01"/>
     <xacro:property name="camera_box_z" value="0.01"/>
-  <xacro:macro name="normal_camera" params="parent_name sensor_name *camera_pose">
+  <xacro:macro name="normal_camera" params="parent_name sensor_name robot_name *camera_pose">
     <link name='${sensor_name}_camera_link'>
-		<!-- <visual>
+		<visual>
 			<origin xyz="0 0 0"
 					rpy="0 0 0"/>
@@ -14,5 +14,5 @@
 				<box size="${camera_box_x} ${camera_box_y} ${camera_box_z}"/>
 			</geometry>
-		</visual> -->
+		</visual>
 	</link>
     <joint name="${sensor_name}_camera_link_joint" type="fixed">
@@ -33,5 +33,5 @@
         <update_rate>10.0</update_rate>
         <camera name="${sensor_name}_SP">
-            <pose>0 0 0 0 0 0</pose>
+            <pose>0.05 0 0 0 0 0</pose>
             <horizontal_fov>1.3962634</horizontal_fov>
             <image>
@@ -46,4 +46,7 @@
         </camera>
         <plugin name="camera_controller" filename="libgazebo_ros_camera.so">
+            <ros>
+                <namespace>/${robot_name}</namespace>
+            </ros>
             <alwaysOn>true</alwaysOn>
             <updateRate>0.0</updateRate>

Commit message: Fix simulated camera

File: nanosaur_gazebo/urdf/nanosaur.urdf.xacro (robot description, xacro)
@@ -28,10 +28,10 @@
     <xacro:if value="${cover_type_name == 'pi'}">
         <xacro:normal_camera parent_name="camera_board" sensor_name="camera" robot_name="nanosaur">
-            <origin xyz="0 0 0" rpy="0 ${M_PI/2} 0" />
+            <origin xyz="0 0 0" rpy="0 -${M_PI/2} 0" />
         </xacro:normal_camera>
     </xacro:if>
     <xacro:if value="${cover_type_name == 'fisheye'}">
         <xacro:wide_angle_camera parent_name="camera_board" sensor_name="camera" robot_name="nanosaur">
-            <origin xyz="0 0 0" rpy="0 0 0" />
+            <origin xyz="0 0 0" rpy="0 -${M_PI/2} 0" />
         </xacro:wide_angle_camera>
     </xacro:if>

File: nanosaur_gazebo/urdf/sensors/camera.gazebo.xacro (robot description, xacro)
@@ -33,5 +33,5 @@
         <update_rate>10.0</update_rate>
         <camera name="${sensor_name}_SP">
-            <pose>0.05 0 0 0 0 0</pose>
+            <pose>0 0 0 0 0 0</pose>
             <horizontal_fov>1.3962634</horizontal_fov>
             <image>

File: nanosaur_gazebo/urdf/sensors/wide.gazebo.xacro (robot description, xacro)
@@ -6,19 +6,19 @@
     <xacro:property name="camera_box_y" value="0.01"/>
     <xacro:property name="camera_box_z" value="0.01"/>
-  <xacro:macro name="wide_angle_camera" params="parent_name sensor_name *camera_pose">
+  <xacro:macro name="wide_angle_camera" params="parent_name sensor_name robot_name *camera_pose">
     <link name='${sensor_name}_camera_link'>
-		<visual>
-			<origin xyz="0 0 0"
-					rpy="0 0 0"/>
-			<geometry>
-				<box size="${camera_box_x} ${camera_box_y} ${camera_box_z}"/>
-			</geometry>
-		</visual>
-	</link>
+      <visual>
+      <origin xyz="0 0 0"
+          rpy="0 0 0"/>
+      <geometry>
+        <box size="${camera_box_x} ${camera_box_y} ${camera_box_z}"/>
+      </geometry>
+      </visual>
+    </link>
     <joint name="${sensor_name}_camera_link_joint" type="fixed">
-		<xacro:insert_block name="camera_pose"/>
-		<parent link="${parent_name}"/>
-		<child link="${sensor_name}_camera_link"/>
-	</joint>
+      <xacro:insert_block name="camera_pose"/>
+      <parent link="${parent_name}"/>
+      <child link="${sensor_name}_camera_link"/>
+    </joint>
     <link name="${sensor_name}_camera_link_frame">
     </link>
@@ -30,5 +30,5 @@
     </joint>
     <gazebo reference="${sensor_name}_camera_link_frame">
-        <sensor name="camera" type="wideanglecamera">
+        <sensor type="wideanglecamera" name="camera">
           <camera>
             <horizontal_fov>6.283</horizontal_fov>

Commit message: Added publish_pointcloud option

File: nanosaur_gazebo/urdf/nanosaur.urdf.xacro (robot description, xacro)
@@ -39,5 +39,5 @@
     </xacro:if>
     <xacro:if value="${cover_type_name == 'realsense'}">
-        <xacro:realsense_camera parent_name="camera_board" sensor_name="camera" robot_name="$(arg robot_name)" />
+        <xacro:realsense_camera parent_name="camera_board" sensor_name="camera" robot_name="$(arg robot_name)" publish_pointcloud="true" />
     </xacro:if>
     <xacro:if value="${cover_type_name == 'zedmini'}">

File: nanosaur_gazebo/urdf/sensors/realsense.gazebo.xacro (robot description, xacro)
@@ -1,8 +1,8 @@
 <?xml version="1.0" ?>
 <robot name="nanosaur_sensor_realsense" xmlns:xacro="http://ros.org/wiki/xacro">
-    <xacro:macro name="realsense_camera" params="parent_name sensor_name robot_name">
+    <xacro:macro name="realsense_camera" params="parent_name sensor_name robot_name publish_pointcloud">
     <gazebo reference="camera_link">
         <sensor name="cameradepth" type="depth">
-            <camera name="camera">
+            <camera name="${sensor_name}">
             <horizontal_fov>1.57</horizontal_fov>
             <image>
@@ -25,5 +25,5 @@
         </sensor>
         <sensor name="cameracolor" type="camera">
-            <camera name="camera">
+            <camera name="${sensor_name}">
                 <horizontal_fov>1.57</horizontal_fov>
                 <image>
@@ -47,5 +47,5 @@
         </sensor>
         <sensor name="cameraired1" type="camera">
-            <camera name="camera">
+            <camera name="${sensor_name}">
                 <horizontal_fov>1.57</horizontal_fov>
                 <image>
@@ -69,5 +69,5 @@
         </sensor>
         <sensor name="cameraired2" type="camera">
-            <camera name="camera">
+            <camera name="${sensor_name}">
                 <horizontal_fov>1.57</horizontal_fov>
                 <image>
@@ -93,5 +93,5 @@
     <gazebo>
         <plugin name="camera" filename="librealsense_gazebo_plugin.so">
-            <prefix>camera</prefix>
+            <prefix>${sensor_name}</prefix>
             <depthUpdateRate>30.0</depthUpdateRate>
             <colorUpdateRate>30.0</colorUpdateRate>
@@ -111,5 +111,5 @@
             <rangeMinDepth>0.3</rangeMinDepth>
             <rangeMaxDepth>3.0</rangeMaxDepth>
-            <pointCloud>true</pointCloud>
+            <pointCloud>${publish_pointcloud}</pointCloud>
             <pointCloudTopicName>depth/color/points</pointCloudTopicName>
             <pointCloudCutoff>0.3</pointCloudCutoff>

Commit message: Fix zed camera

File: nanosaur_gazebo/urdf/nanosaur.urdf.xacro (robot description, xacro)
@@ -6,4 +6,5 @@
     <xacro:include filename="$(find nanosaur_gazebo)/urdf/diff_drive.gazebo.xacro" />
     <!-- Sensors -->
+    <xacro:include filename="$(find nanosaur_gazebo)/urdf/sensors/imu.gazebo.xacro" />
     <xacro:include filename="$(find nanosaur_gazebo)/urdf/sensors/camera.gazebo.xacro" />
     <xacro:include filename="$(find nanosaur_gazebo)/urdf/sensors/wide.gazebo.xacro" />
@@ -15,5 +16,5 @@
     <xacro:property name="cover_type_name" value="$(arg cover_type)" />
     <xacro:arg name="depth_camera"  default="left"/>
-    <xacro:arg name="resolution"    default="HD720"/>
+    <xacro:arg name="resolution"    default="VGA"/>
     <!-- nanosaur robot
          "diff_drive_emulation" parameter enable simulation mode.
@@ -44,6 +45,6 @@
         <xacro:realsense_camera parent_name="camera_board" sensor_name="camera" robot_name="$(arg robot_name)" publish_pointcloud="true" />
     </xacro:if>
-    <xacro:if value="${cover_type_name == 'zedmini'}">
-        <xacro:zed_gazebo_camera sensor_name="camera" robot_name="$(arg robot_name)"
+    <xacro:if value="${cover_type_name == 'zed'}">
+        <xacro:zed_gazebo_camera parent_name="camera_board" sensor_name="zed" robot_name="$(arg robot_name)"
             camera_model="zedm" depth_camera="$(arg depth_camera)" resolution="$(arg resolution)" />
     </xacro:if>

File: nanosaur_gazebo/urdf/sensors/zed.gazebo.xacro (robot description, xacro)
@@ -2,4 +2,18 @@
 <robot name="nanosaur_sensor_zed" xmlns:xacro="http://ros.org/wiki/xacro">
     <xacro:macro name="zed_gazebo_camera" params="parent_name sensor_name robot_name camera_model depth_camera resolution">
+        <link name="${camera_model}_${depth_camera}_depth_frame" />
+        <joint name="${sensor_name}_depth_gazebo_joint" type="fixed">
+            <origin xyz="0 0 0" rpy="0 0 0" />
+            <parent link="${camera_model}_${depth_camera}_camera_frame" />
+            <child link="${camera_model}_${depth_camera}_depth_frame" />
+        </joint>
+        <xacro:if value="${camera_model == 'zedm'}">
+          <link name="${sensor_name}_imu_frame_gazebo" />
+          <joint name="${sensor_name}_imu_gazebo_joint" type="fixed">
+              <origin xyz="0 0 0" rpy="0 0 0" />
+              <parent link="${camera_model}_camera_center" />
+              <child link="${sensor_name}_imu_frame_gazebo" />
+          </joint>
+        </xacro:if>
         <xacro:property name="depth_rate" value="30" />
         <xacro:if value="${resolution == 'HD2K'}">
@@ -18,7 +32,12 @@
             <xacro:property name="update_rate" value="60" />
         </xacro:if>
-        <xacro:if value="${resolution == 'VGA'}">
+        <xacro:if value="${resolution == 'WVGA'}">
             <xacro:property name="resolution_width" value="1344" />
             <xacro:property name="resolution_heigth" value="376" />
+            <xacro:property name="update_rate" value="100" />
+        </xacro:if>
+        <xacro:if value="${resolution == 'VGA'}">
+            <xacro:property name="resolution_width" value="640" />
+            <xacro:property name="resolution_heigth" value="480" />
             <xacro:property name="update_rate" value="100" />
         </xacro:if>
@@ -28,20 +47,12 @@
             <xacro:property name="clip_near" value="0.3" />
             <xacro:property name="clip_far" value="25" />
-            <!-- Gazebo color -->
-            <gazebo reference="${camera_model}_camera_center">
-            <material>Gazebo/Grey</material>
-            </gazebo>
         </xacro:if>
         <xacro:if value="${camera_model == 'zedm'}">
-            <xacro:property name="baseline" value="0.06" />
+            <xacro:property name="baseline" value="0.063" />
             <xacro:property name="fov" value="2.0" />
             <xacro:property name="clip_near" value="0.1" />
             <xacro:property name="clip_far" value="15" />
             <!-- Add IMU for ZED -->
-            <xacro:imu_gazebo name="${camera_name}" frame="${camera_name}_imu_frame_gazebo" />
-            <!-- Gazebo color -->
-            <gazebo reference="${camera_model}_camera_center">
-            <material>Gazebo/DarkGrey</material>
-            </gazebo>
+            <!-- <xacro:imu_gazebo name="${sensor_name}" frame="${sensor_name}_imu_frame_gazebo" /> -->
         </xacro:if>
         <xacro:if value="${camera_model == 'zed2'}">
@@ -51,106 +62,75 @@
             <xacro:property name="clip_far" value="20" />
             <!-- Add IMU for ZED -->
-            <xacro:imu_gazebo name="${camera_name}" frame="${camera_name}_imu_frame_gazebo" />
-            <!-- Gazebo color -->
-            <gazebo reference="${camera_model}_camera_center">
-            <material>Gazebo/Black</material>
-            </gazebo>
+            <xacro:imu_gazebo name="${sensor_name}" frame="${sensor_name}_imu_frame_gazebo" />
         </xacro:if>
-        <gazebo reference="${camera_model}_camera_center">
-            <sensor type="multicamera" name="${camera_name}_stereo_camera">
-                <update_rate>${update_rate}</update_rate>
-                <camera name="left">
-                    <horizontal_fov>${fov}</horizontal_fov>
-                    <image>
-                        <width>${resolution_width}</width>
-                        <height>${resolution_heigth}</height>
-                        <format>R8G8B8</format>
-                    </image>
-                    <clip>
-                        <near>0.02</near>
-                        <far>300</far>
-                    </clip>
-                    <noise>
-                        <type>gaussian</type>
-                        <mean>0.0</mean>
-                        <stddev>0.007</stddev>
-                    </noise>
-                </camera>
-                <camera name="right">
-                    <horizontal_fov>${fov}</horizontal_fov>
-                    <image>
-                        <width>${resolution_width}</width>
-                        <height>${resolution_heigth}</height>
-                        <format>R8G8B8</format>
-                    </image>
-                    <clip>
-                        <near>0.02</near>
-                        <far>300</far>
-                    </clip>
-                    <noise>
-                        <type>gaussian</type>
-                        <mean>0.0</mean>
-                        <stddev>0.007</stddev>
-                    </noise>
-                </camera>
-                <plugin name="stereo_camera_controller" filename="libgazebo_ros_multicamera.so">
-                    <cameraName>${camera_name}</cameraName>
-                    <alwaysOn>true</alwaysOn>
-                    <updateRate>${update_rate}</updateRate>
-                    <imageTopicName>image_rect_color</imageTopicName>
-                    <cameraInfoTopicName>camera_info</cameraInfoTopicName>
-                    <frameName>${camera_model}_left_camera_optical_frame</frameName>
-                    <!--<rightFrameName>${camera_model}_right_camera_optical_frame</rightFrameName>-->
-                    <baseline>${baseline}</baseline>
-                    <distortionK1>0.0</distortionK1>
-                    <distortionK2>0.0</distortionK2>
-                    <distortionK3>0.0</distortionK3>
-                    <distortionT1>0.0</distortionT1>
-                    <distortionT2>0.0</distortionT2>
-                    <hackBaseline>0.07</hackBaseline>
-                </plugin>
-            </sensor>
-        </gazebo>
-        <gazebo reference="${camera_model}_camera_center">
-            <sensor type="depth" name="${camera_name}_depth">
-                <always_on>true</always_on>
-                <update_rate>${depth_rate}</update_rate>
-                <camera>
-                    <horizontal_fov>${fov}</horizontal_fov>
-                    <image>
-                        <format>R8G8B8</format>
-                        <width>${resolution_width}</width>
-                        <height>${resolution_heigth}</height>
-                    </image>
-                    <clip>
-                        <near>${clip_near}</near>
-                        <far>${clip_far}</far>
-                    </clip>
-                </camera>
-                <plugin name="${camera_name}_camera_controller" filename="libgazebo_ros_openni_kinect.so">
-                    <cameraName>${camera_name}</cameraName>
-                    <alwaysOn>true</alwaysOn>
-                    <updateRate>${depth_rate}</updateRate>
-                    <imageTopicName>rgb/image_rect_color</imageTopicName>
-                    <depthImageTopicName>depth/depth_registered</depthImageTopicName>
-                    <pointCloudTopicName>depth/points</pointCloudTopicName>
-                    <cameraInfoTopicName>rgb/camera_info</cameraInfoTopicName>
-                    <depthImageCameraInfoTopicName>depth/camera_info</depthImageCameraInfoTopicName>
-                    <frameName>camera_depth_frame_gazebo</frameName>
-                    <baseline>${baseline}</baseline>
-                    <pointCloudCutoff>0.02</pointCloudCutoff>
-                    <distortionK1>0</distortionK1>
-                    <distortionK2>0</distortionK2>
-                    <distortionK3>0</distortionK3>
-                    <distortionT1>0</distortionT1>
-                    <distortionT2>0</distortionT2>
-                    <CxPrime>0</CxPrime>
-                    <Cx>0</Cx>
-                    <Cy>0</Cy>
-                    <focalLength>0</focalLength>
-                    <hackBaseline>0</hackBaseline>
-                </plugin>
-            </sensor>
-        </gazebo>
+      <gazebo reference="${camera_model}_${depth_camera}_depth_frame">
+        <sensor type="depth" name="${sensor_name}/left">
+          <update_rate>${depth_rate}</update_rate>
+          <visualize>1</visualize>
+          <camera>
+            <pose>0 0 0 0 0 0</pose>
+            <horizontal_fov>${fov}</horizontal_fov>
+            <image>
+              <width>${resolution_width}</width>
+              <height>${resolution_heigth}</height>
+              <format>B8G8R8</format>
+            </image>
+            <depth_camera>
+            </depth_camera>
+            <clip>
+              <near>0.02</near>
+              <far>300</far>
+            </clip>
+            <noise>
+              <type>gaussian</type>
+              <!-- Noise is sampled independently per pixel on each frame.
+                   That pixel's noise value is added to each of its color
+                   channels, which at that point lie in the range [0,1]. -->
+              <mean>0.0</mean>
+              <stddev>0.007</stddev>
+            </noise>
+          </camera>
+          <plugin name="${camera_model}_left_controller" filename="libgazebo_ros_camera.so">
+            <ros>
+                <namespace>/${robot_name}</namespace>
+            </ros>
+            <alwaysOn>true</alwaysOn>
+            <updateRate>0.0</updateRate>
+            <cameraName>${sensor_name}/left</cameraName>
+            <frameName>${camera_model}_left_camera_frame</frameName>
+            <min_depth>${clip_near}</min_depth>
+            <max_depth>${clip_far}</max_depth>
+          </plugin>
+        </sensor>
+      </gazebo>
+    <gazebo reference="${camera_model}_right_camera_frame">
+        <sensor type="camera" name="${sensor_name}/right">
+        <update_rate>${update_rate}</update_rate>
+        <camera name="${sensor_name}/right">
+            <pose>0 0 0 0 0 0</pose>
+            <horizontal_fov>${fov}</horizontal_fov>
+            <image>
+              <width>${resolution_width}</width>
+              <height>${resolution_heigth}</height>
+              <format>R8G8B8</format>
+            </image>
+            <clip>
+              <near>0.02</near>
+              <far>300</far>
+            </clip>
+        </camera>
+        <plugin name="${camera_model}_right_controller" filename="libgazebo_ros_camera.so">
+            <ros>
+                <namespace>/${robot_name}</namespace>
+            </ros>
+            <alwaysOn>true</alwaysOn>
+            <updateRate>0.0</updateRate>
+            <cameraName>${sensor_name}</cameraName>
+            <imageTopicName>image_raw</imageTopicName>
+            <cameraInfoTopicName>camera_info</cameraInfoTopicName>
+            <frameName>${camera_model}_right_camera_frame</frameName>
+        </plugin>
+        </sensor>
+    </gazebo>
     </xacro:macro>
 </robot>
