Commit message: improve gazebo launcher

File: nanosaur_gazebo/urdf/diff_drive.gazebo.xacro (robot description, xacro)
@@ -1,29 +1,43 @@
 <?xml version="1.0"?>
 <robot name="nanosaur_track" xmlns:xacro="http://ros.org/wiki/xacro">
-    <xacro:macro name="track_drive" params="parent robot_name">
+    <!--Reference http://gazebosim.org/tutorials?tut=ros_gzplugins#DifferentialDrive -->
+    <xacro:macro name="track_drive" params="parent robot_name update_rate wheel_radius wheel_separation">
         <gazebo>
             <plugin filename="libgazebo_ros_diff_drive.so" name="skid_steer_drive_controller">
             <ros>
                 <namespace>/${robot_name}</namespace>
-                <argument>/cmd_vel:=cmd_vel</argument>
-                <argument>/odom:=odom</argument>
+                <argument>--ros-args --remap /cmd_vel:=cmd_vel</argument>
+                <argument>--ros-args --remap /odom:=odom</argument>
             </ros>
-            <update_rate>100.0</update_rate>
+            <!-- Plugin update rate in Hz -->
+            <update_rate>${update_rate}</update_rate>
             <num_wheel_pairs>2</num_wheel_pairs>
-            <odometry_frame>odom</odometry_frame>
+            <!-- Name of left joint, defaults to `left_joint` -->
             <left_joint>sprocket_left_joint</left_joint>
             <left_joint>wheel_left_joint</left_joint>
-            <wheel_separation>0.4</wheel_separation>
-            <wheel_diameter>0.2</wheel_diameter>
+            <!-- Name of right joint, defaults to `right_joint` -->
             <right_joint>sprocket_right_joint</right_joint>
             <right_joint>wheel_right_joint</right_joint>
-            <wheel_separation>0.4</wheel_separation>
-            <wheel_diameter>0.2</wheel_diameter>
+            <!-- The distance from the center of one wheel to the other, in meters, defaults to 0.34 m -->
+            <wheel_separation>${wheel_separation}</wheel_separation>
+            <!-- Diameter of the wheels, in meters, defaults to 0.15 m -->
+            <wheel_diameter>${wheel_radius * 2}</wheel_diameter>
+            <!-- Wheel acceleration, in rad/s^2, defaults to 0.0 rad/s^2 -->
+            <wheel_acceleration>0.0</wheel_acceleration>
+            <!-- Maximum torque which the wheels can produce, in Nm, defaults to 5 Nm -->
+            <max_wheel_torque>15</max_wheel_torque>
+            <!-- Odometry frame, defaults to `odom` -->
+            <odometry_frame>odom</odometry_frame>
+            <!-- Robot frame to calculate odometry from, defaults to `base_footprint` -->
             <robot_base_frame>${parent}</robot_base_frame>
-            <max_wheel_torque>15</max_wheel_torque>
+            <!-- Set to true to publish transforms for the odometry, defaults to true -->
             <publish_odom>true</publish_odom>
             <publish_odom_tf>true</publish_odom_tf>
+            <!-- Set to true to publish transforms for the wheel links, defaults to false -->
             <publish_wheel_tf>true</publish_wheel_tf>
-            <odometry_source>world</odometry_source>
+            <!-- Odometry source, 0 for ENCODER, 1 for WORLD, defaults to WORLD -->
+            <odometry_source>1</odometry_source>
+            <!-- Set to true to publish sensor_msgs/JointState on /joint_states for the wheel joints, defaults to false -->
+            <publis_wheel_joint_state>false</publis_wheel_joint_state>
             </plugin>
         </gazebo>

File: nanosaur_gazebo/urdf/nanosaur.urdf.xacro (robot description, xacro)
@@ -8,10 +8,14 @@
     <xacro:arg name="cover_type" default="realsense" /> <!--options: pi, fisheye, realsense, zedmini -->
     <!-- nanosaur robot
-         "simulation" parameter enable simulation mode.
+         "diff_drive_emulation" parameter enable simulation mode.
          Add extra wheel and center sprocket for differential drive simulation -->
     <xacro:nanosaur cover_type="$(arg cover_type)"
                     use_nominal_extrinsics="true"
-                    simulation="true" />
+                    diff_drive_emulation="true" />
     <!-- nanosaur differential drive controller -->
-    <xacro:track_drive parent="base_link" robot_name="nanosaur"/>
+    <xacro:track_drive parent="base_link"
+                       robot_name="nanosaur"
+                       update_rate="100.0"
+                       wheel_radius="0.0150"
+                       wheel_separation="0.4" />
 </robot>

Commit message: Improve gazebo simulation

File: nanosaur_gazebo/urdf/diff_drive.gazebo.xacro (robot description, xacro)
@@ -2,5 +2,5 @@
 <robot name="nanosaur_track" xmlns:xacro="http://ros.org/wiki/xacro">
     <!--Reference http://gazebosim.org/tutorials?tut=ros_gzplugins#DifferentialDrive -->
-    <xacro:macro name="track_drive" params="parent robot_name update_rate wheel_radius wheel_separation">
+    <xacro:macro name="track_drive" params="parent robot_name update_rate wheel_radius wheel_separation publish_odom_tf">
         <gazebo>
             <plugin filename="libgazebo_ros_diff_drive.so" name="skid_steer_drive_controller">
@@ -33,5 +33,5 @@
             <!-- Set to true to publish transforms for the odometry, defaults to true -->
             <publish_odom>true</publish_odom>
-            <publish_odom_tf>true</publish_odom_tf>
+            <publish_odom_tf>${publish_odom_tf}</publish_odom_tf>
             <!-- Set to true to publish transforms for the wheel links, defaults to false -->
             <publish_wheel_tf>true</publish_wheel_tf>

File: nanosaur_gazebo/urdf/nanosaur.urdf.xacro (robot description, xacro)
@@ -16,4 +16,5 @@
     <xacro:property name="cover_type_name" value="$(arg cover_type)" />
     <xacro:arg name="publish_pointcloud"  default="false"/>
+    <xacro:arg name="publish_odom_tf"  default="false"/>
     <xacro:arg name="depth_camera"  default="left"/>
     <xacro:arg name="resolution"    default="VGA"/>
@@ -31,5 +32,6 @@
                        update_rate="100.0"
                        wheel_radius="0.0150"
-                       wheel_separation="0.4" />
+                       wheel_separation="0.4"
+                       publish_odom_tf="$(arg publish_odom_tf)" />
     <!-- Nanosaur sensors -->
     <xacro:if value="${cover_type_name == 'pi'}">
