Commit message: minor fixes and bug #2

File: nanosaur_gazebo/urdf/sensors/zed.gazebo.xacro (robot description, xacro)
@@ -45,12 +45,12 @@
             <xacro:property name="baseline" value="0.12" />
             <xacro:property name="fov" value="2.0" />
-            <xacro:property name="clip_near" value="0.3" />
-            <xacro:property name="clip_far" value="25" />
+            <xacro:property name="min_depth" value="0.3" />
+            <xacro:property name="max_depth" value="25" />
         </xacro:if>
         <xacro:if value="${camera_model == 'zedm'}">
             <xacro:property name="baseline" value="0.063" />
             <xacro:property name="fov" value="2.0" />
-            <xacro:property name="clip_near" value="0.1" />
-            <xacro:property name="clip_far" value="15" />
+            <xacro:property name="min_depth" value="0.1" />
+            <xacro:property name="max_depth" value="15" />
             <!-- Add IMU for ZED -->
             <!-- <xacro:imu_gazebo name="${sensor_name}" frame="${sensor_name}_imu_frame_gazebo" /> -->
@@ -59,6 +59,6 @@
             <xacro:property name="baseline" value="0.12" />
             <xacro:property name="fov" value="1.8" />
-            <xacro:property name="clip_near" value="0.2" />
-            <xacro:property name="clip_far" value="20" />
+            <xacro:property name="min_depth" value="0.2" />
+            <xacro:property name="max_depth" value="20" />
             <!-- Add IMU for ZED -->
             <xacro:imu_gazebo name="${sensor_name}" frame="${sensor_name}_imu_frame_gazebo" />
@@ -99,6 +99,6 @@
             <cameraName>${sensor_name}/left</cameraName>
             <frameName>${camera_model}_left_camera_frame</frameName>
-            <min_depth>${clip_near}</min_depth>
-            <max_depth>${clip_far}</max_depth>
+            <min_depth>${min_depth}</min_depth>
+            <max_depth>${max_depth}</max_depth>
           </plugin>
         </sensor>
