Commit message: Fix realsense camera

File: nanosaur_gazebo/urdf/sensors/realsense.gazebo.xacro (robot description, xacro)
@@ -2,118 +2,68 @@
 <robot name="nanosaur_sensor_realsense" xmlns:xacro="http://ros.org/wiki/xacro">
     <xacro:macro name="realsense_camera" params="parent_name sensor_name robot_name publish_pointcloud">
-    <gazebo reference="camera_link">
-        <sensor name="cameradepth" type="depth">
-            <camera name="${sensor_name}">
-            <horizontal_fov>1.57</horizontal_fov>
-            <image>
-                <width>1280</width>
-                <height>720</height>
-            </image>
-            <clip>
-                <near>0.1</near>
-                <far>100</far>
-            </clip>
-            <noise>
-                <type>gaussian</type>
-                <mean>0.0</mean>
-                <stddev>0.100</stddev>
-            </noise>
-            </camera>
-            <always_on>1</always_on>
-            <update_rate>30</update_rate>
-            <visualize>0</visualize>
-        </sensor>
-        <sensor name="cameracolor" type="camera">
-            <camera name="${sensor_name}">
-                <horizontal_fov>1.57</horizontal_fov>
-                <image>
-                    <width>1280</width>
-                    <height>720</height>
-                    <format>RGB_INT8</format>
-                </image>
-                <clip>
-                    <near>0.1</near>
-                    <far>100</far>
-                </clip>
-                <noise>
-                    <type>gaussian</type>
-                    <mean>0.0</mean>
-                    <stddev>0.007</stddev>
-                </noise>
-            </camera>
-            <always_on>1</always_on>
-            <update_rate>30</update_rate>
-            <visualize>1</visualize>
-        </sensor>
-        <sensor name="cameraired1" type="camera">
-            <camera name="${sensor_name}">
-                <horizontal_fov>1.57</horizontal_fov>
-                <image>
-                    <width>1280</width>
-                    <height>720</height>
-                    <format>L_INT8</format>
-                </image>
-                <clip>
-                    <near>0.1</near>
-                    <far>100</far>
-                </clip>
-                <noise>
-                    <type>gaussian</type>
-                    <mean>0.0</mean>
-                    <stddev>0.05</stddev>
-                </noise>
-            </camera>
-            <always_on>1</always_on>
-            <update_rate>1</update_rate>
-            <visualize>0</visualize>
-        </sensor>
-        <sensor name="cameraired2" type="camera">
-            <camera name="${sensor_name}">
-                <horizontal_fov>1.57</horizontal_fov>
-                <image>
-                    <width>1280</width>
-                    <height>720</height>
-                    <format>L_INT8</format>
-                </image>
-                <clip>
-                    <near>0.1</near>
-                    <far>100</far>
-                </clip>
-                <noise>
-                    <type>gaussian</type>
-                    <mean>0.0</mean>
-                    <stddev>0.05</stddev>
-                </noise>
-            </camera>
-            <always_on>1</always_on>
-            <update_rate>1</update_rate>
-            <visualize>0</visualize>
-        </sensor>
-    </gazebo>
-    <gazebo>
-        <plugin name="camera" filename="librealsense_gazebo_plugin.so">
-            <prefix>${sensor_name}</prefix>
-            <depthUpdateRate>30.0</depthUpdateRate>
-            <colorUpdateRate>30.0</colorUpdateRate>
-            <infraredUpdateRate>1.0</infraredUpdateRate>
-            <depthTopicName>${robot_name}/${sensor_name}/aligned_depth_to_color/image_raw</depthTopicName>
-            <depthCameraInfoTopicName>${robot_name}/${sensor_name}/depth/camera_info</depthCameraInfoTopicName>
-            <colorTopicName>${robot_name}/${sensor_name}/color/image_raw</colorTopicName>
-            <colorCameraInfoTopicName>${robot_name}/${sensor_name}/color/camera_info</colorCameraInfoTopicName>
-            <infrared1TopicName>${robot_name}/${sensor_name}/infra1/image_raw</infrared1TopicName>
-            <infrared1CameraInfoTopicName>${robot_name}/${sensor_name}/infra1/camera_info</infrared1CameraInfoTopicName>
-            <infrared2TopicName>${robot_name}/${sensor_name}/infra2/image_raw</infrared2TopicName>
-            <infrared2CameraInfoTopicName>${robot_name}/${sensor_name}/infra2/camera_info</infrared2CameraInfoTopicName>
-            <colorOpticalframeName>camera_color_optical_frame</colorOpticalframeName>
-            <depthOpticalframeName>camera_depth_optical_frame</depthOpticalframeName>
-            <infrared1OpticalframeName>camera_infra1_optical_frame</infrared1OpticalframeName>
-            <infrared2OpticalframeName>camera_infra2_optical_frame</infrared2OpticalframeName>
-            <rangeMinDepth>0.3</rangeMinDepth>
-            <rangeMaxDepth>3.0</rangeMaxDepth>
-            <pointCloud>${publish_pointcloud}</pointCloud>
-            <pointCloudTopicName>${robot_name}/${sensor_name}/depth/color/points</pointCloudTopicName>
-            <pointCloudCutoff>0.3</pointCloudCutoff>
-        </plugin>
-    </gazebo>
+        <xacro:property name="update_rate" value="30" />
+        <xacro:property name="resolution_width" value="640" />
+        <xacro:property name="resolution_heigth" value="480" />
+        <xacro:property name="fov" value="1.57" />
+        <xacro:property name="baseline" value="0.05" />
+        <gazebo reference="camera_infra1_frame">
+            <sensor type="multicamera" name="${sensor_name}">
+                <pose>0 0 0 0 0 0</pose>
+                <update_rate>${update_rate}</update_rate>
+                <visualize>true</visualize>
+                <camera name="infra1">
+                    <horizontal_fov>${fov}</horizontal_fov>
+                    <image>
+                        <width>${resolution_width}</width>
+                        <height>${resolution_heigth}</height>
+                        <format>R8G8B8</format>
+                    </image>
+                    <clip>
+                        <near>0.02</near>
+                        <far>300</far>
+                    </clip>
+                    <noise>
+                        <type>gaussian</type>
+                        <!-- Noise is sampled independently per pixel on each frame.
+                            That pixel's noise value is added to each of its color
+                            channels, which at that point lie in the range [0,1]. -->
+                        <mean>0.0</mean>
+                        <stddev>0.007</stddev>
+                    </noise>
+                </camera>
+                <camera name="infra2">
+                    <pose>0 -${baseline} 0 0 0 0</pose>
+                    <horizontal_fov>${fov}</horizontal_fov>
+                    <image>
+                        <width>${resolution_width}</width>
+                        <height>${resolution_heigth}</height>
+                        <format>R8G8B8</format>
+                    </image>
+                    <clip>
+                        <near>0.02</near>
+                        <far>300</far>
+                    </clip>
+                    <noise>
+                        <type>gaussian</type>
+                        <!-- Noise is sampled independently per pixel on each frame.
+                            That pixel's noise value is added to each of its color
+                            channels, which at that point lie in the range [0,1]. -->
+                        <mean>0.0</mean>
+                        <stddev>0.007</stddev>
+                    </noise>
+                </camera>
+                <plugin name="camera_controller" filename="libgazebo_ros_camera.so">
+                    <ros>
+                        <namespace>/${robot_name}</namespace>
+                    </ros>
+                    <alwaysOn>true</alwaysOn>
+                    <updateRate>0.0</updateRate>
+                    <cameraName>${sensor_name}</cameraName>
+                    <imageTopicName>image_raw</imageTopicName>
+                    <cameraInfoTopicName>camera_info</cameraInfoTopicName>
+                    <frameName>camera_infra1_optical_frame</frameName>
+                </plugin>
+            </sensor>
+        </gazebo>
     </xacro:macro>
 </robot>
