Commit message: Add joint state controller

File: nanosaur_ignition/urdf/diff_drive.ignition.xacro (robot description, xacro)
@@ -1,45 +1,49 @@
 <?xml version="1.0"?>
-<robot name="nanosaur_track" xmlns:xacro="http://ros.org/wiki/xacro">
-        <!-- reference
+<robot name="nanosaur_track"
+    xmlns:xacro="http://ros.org/wiki/xacro">
+    <!-- reference
             https://github.com/gazebosim/gz-sim/blob/5b21ec87306c35b3494adc25694fac8b8d1bb7de/src/systems/diff_drive/DiffDrive.hh#L57
             https://github.com/Blast545/ign_tutorials
         -->
-        <xacro:macro name="track_drive" params="parent robot_name update_rate wheel_radius wheel_separation publish_odom_tf">
+    <xacro:macro name="track_drive" params="parent robot_name update_rate wheel_radius wheel_separation publish_odom_tf">
         <gazebo>
             <plugin name="ignition::gazebo::systems::DiffDrive" filename="libignition-gazebo-diff-drive-system.so">
-            <!-- Plugin update rate in Hz -->
-            <update_rate>${update_rate}</update_rate>
-            <num_wheel_pairs>2</num_wheel_pairs>
-            <!-- Name of left joint, defaults to `left_joint` -->
-            <left_joint>sprocket_left_joint</left_joint>
-            <left_joint>wheel_left_joint</left_joint>
-            <!-- Name of right joint, defaults to `right_joint` -->
-            <right_joint>sprocket_right_joint</right_joint>
-            <right_joint>wheel_right_joint</right_joint>
-            <!-- The distance from the center of one wheel to the other, in meters, defaults to 0.34 m -->
-            <wheel_separation>${wheel_separation}</wheel_separation>
-            <!-- Diameter of the wheels, in meters, defaults to 0.15 m -->
-            <wheel_diameter>${wheel_radius * 2}</wheel_diameter>
-            <!-- Wheel acceleration, in rad/s^2, defaults to 0.0 rad/s^2 -->
-            <wheel_acceleration>0.0</wheel_acceleration>
-            <!-- Maximum torque which the wheels can produce, in Nm, defaults to 5 Nm -->
-            <max_wheel_torque>15</max_wheel_torque>
-            <!-- Odometry frame, defaults to `odom` -->
-            <odometry_frame>odom</odometry_frame>
-            <!-- Robot frame to calculate odometry from, defaults to `base_footprint` -->
-            <robot_base_frame>${parent}</robot_base_frame>
-            <!-- Set to true to publish transforms for the odometry, defaults to true -->
-            <publish_odom>true</publish_odom>
-            <publish_odom_tf>${publish_odom_tf}</publish_odom_tf>
-            <!-- Set to true to publish transforms for the wheel links, defaults to false -->
-            <publish_wheel_tf>true</publish_wheel_tf>
-            <!-- Odometry source, 0 for ENCODER, 1 for WORLD, defaults to WORLD -->
-            <odometry_source>1</odometry_source>
-            <!-- Set to true to publish sensor_msgs/JointState on /joint_states for the wheel joints, defaults to false -->
-            <publis_wheel_joint_state>false</publis_wheel_joint_state>
-            <!-- Custom topic that this system will subscribe to in order to
+                <!-- Plugin update rate in Hz -->
+                <update_rate>${update_rate}</update_rate>
+                <num_wheel_pairs>2</num_wheel_pairs>
+                <!-- Name of left joint, defaults to `left_joint` -->
+                <left_joint>sprocket_left_joint</left_joint>
+                <left_joint>wheel_left_joint</left_joint>
+                <!-- Name of right joint, defaults to `right_joint` -->
+                <right_joint>sprocket_right_joint</right_joint>
+                <right_joint>wheel_right_joint</right_joint>
+                <!-- The distance from the center of one wheel to the other, in meters, defaults to 0.34 m -->
+                <wheel_separation>${wheel_separation}</wheel_separation>
+                <!-- Diameter of the wheels, in meters, defaults to 0.15 m -->
+                <wheel_radius>${wheel_radius}</wheel_radius>
+                <!-- Wheel acceleration, in rad/s^2, defaults to 0.0 rad/s^2 -->
+                <wheel_acceleration>0.0</wheel_acceleration>
+                <!-- Maximum torque which the wheels can produce, in Nm, defaults to 5 Nm -->
+                <max_wheel_torque>15</max_wheel_torque>
+                <!-- Odometry frame, defaults to `odom` -->
+                <odometry_frame>odom</odometry_frame>
+                <!-- Robot frame to calculate odometry from, defaults to `base_footprint` -->
+                <robot_base_frame>${parent}</robot_base_frame>
+                <!-- Set to true to publish transforms for the odometry, defaults to true -->
+                <publish_odom>true</publish_odom>
+                <publish_odom_tf>${publish_odom_tf}</publish_odom_tf>
+                <!-- Set to true to publish transforms for the wheel links, defaults to false -->
+                <publish_wheel_tf>true</publish_wheel_tf>
+                <!-- Odometry source, 0 for ENCODER, 1 for WORLD, defaults to WORLD -->
+                <odometry_source>1</odometry_source>
+                <!-- Set to true to publish sensor_msgs/JointState on /joint_states for the wheel joints, defaults to false -->
+                <publish_wheel_joint_state>true</publish_wheel_joint_state>
+                <!-- Custom topic that this system will subscribe to in order to
                  receive command velocity messages. This element if optional, and the
                  default value is /model/{name_of_model}/cmd_vel -->
-            <topic>cmd_vel</topic>
+                <topic>cmd_vel</topic>
+            </plugin>
+            <!-- Joint states plugin -->
+            <plugin name="ignition::gazebo::systems::JointStatePublisher" filename="libignition-gazebo-joint-state-publisher-system.so">
             </plugin>
         </gazebo>
