Commit message: Add cmd_vel emulation and camera driver

File: nanosaur_ignition/urdf/nanosaur.ignition.xacro (robot description, xacro)
@@ -4,5 +4,7 @@
     <xacro:include filename="$(find nanosaur_description)/urdf/robot.urdf.xacro" />
     <!-- differential drive -->
-    <xacro:include filename="$(find nanosaur_ignition)/urdf/diff_drive.gazebo.xacro" />
+    <xacro:include filename="$(find nanosaur_ignition)/urdf/diff_drive.ignition.xacro" />
+    <!-- Sensors -->
+    <xacro:include filename="$(find nanosaur_ignition)/urdf/sensors/camera.ignition.xacro" />
     <xacro:arg name="robot_name" default="nanosaur" />
     <!-- camera definitions -->
@@ -30,4 +32,7 @@
     <!-- Nanosaur sensors -->
     <xacro:if value="${cover_type_name == 'pi'}">
+        <xacro:normal_camera parent_name="camera_board" sensor_name="camera" robot_name="$(arg robot_name)">
+            <origin xyz="0 0 0" rpy="0 -${M_PI/2} 0" />
+        </xacro:normal_camera>
     </xacro:if>
     <xacro:if value="${cover_type_name == 'fisheye'}">

Commit message: Improved nanosaur ignition with ros2 control

File: nanosaur_ignition/urdf/nanosaur.ignition.xacro (robot description, xacro)
@@ -5,4 +5,5 @@
     <!-- differential drive -->
     <xacro:include filename="$(find nanosaur_ignition)/urdf/diff_drive.ignition.xacro" />
+    <xacro:include filename="$(find nanosaur_ignition)/urdf/ros2_control.ignition.xacro" />
     <!-- Sensors -->
     <xacro:include filename="$(find nanosaur_ignition)/urdf/sensors/camera.ignition.xacro" />
@@ -12,4 +13,6 @@
     <xacro:arg name="cover_type" default="fisheye" /> <!--options: pi, fisheye, realsense, zedmini -->
     <xacro:property name="cover_type_name" value="$(arg cover_type)" />
+    <!-- control definitions -->
+    <xacro:property name="control_type_name" value="ros2_control" /> <!--options: ros2_control, diff_drive -->
     <xacro:arg name="publish_pointcloud"  default="false"/>
     <xacro:arg name="publish_odom_tf"  default="false"/>
@@ -22,13 +25,17 @@
     <xacro:nanosaur cover_type="$(arg cover_type)"
                     use_nominal_extrinsics="true"
-                    diff_drive_emulation="true"
-                    path_meshes="file://$(find nanosaur_description)/meshes" />
+                    diff_drive_emulation="true"/>
+    <xacro:if value="${control_type_name == 'ros2_control'}">
+        <xacro:nanosaur_ros2_control/>
+    </xacro:if>
     <!-- nanosaur differential drive controller -->
-    <xacro:track_drive parent="base_link"
-                       robot_name="$(arg robot_name)"
-                       update_rate="100.0"
-                       wheel_radius="0.0150"
-                       wheel_separation="0.4"
-                       publish_odom_tf="$(arg publish_odom_tf)" />
+    <xacro:if value="${control_type_name == 'diff_drive'}">
+        <xacro:track_drive parent="base_link"
+                        robot_name="$(arg robot_name)"
+                        update_rate="100.0"
+                        wheel_radius="0.0150"
+                        wheel_separation="0.4"
+                        publish_odom_tf="$(arg publish_odom_tf)" />
+    </xacro:if>
     <!-- Nanosaur sensors -->
     <xacro:if value="${cover_type_name == 'pi'}">

Commit message: Minor improvements

File: nanosaur_ignition/urdf/nanosaur.ignition.xacro (robot description, xacro)
@@ -11,8 +11,8 @@
     <xacro:arg name="robot_name" default="nanosaur" />
     <!-- camera definitions -->
-    <xacro:arg name="cover_type" default="fisheye" /> <!--options: pi, fisheye, realsense, zedmini -->
+    <xacro:arg name="cover_type" default="fisheye" /> <!--options pi, fisheye, realsense, zedmini -->
     <xacro:property name="cover_type_name" value="$(arg cover_type)" />
     <!-- control definitions -->
-    <xacro:property name="control_type_name" value="ros2_control" /> <!--options: ros2_control, diff_drive -->
+    <xacro:property name="control_type_name" value="ros2_control" /> <!--options ros2_control, diff_drive -->
     <xacro:arg name="publish_pointcloud"  default="false"/>
     <xacro:arg name="publish_odom_tf"  default="false"/>
@@ -27,5 +27,5 @@
                     diff_drive_emulation="true"/>
     <xacro:if value="${control_type_name == 'ros2_control'}">
-        <xacro:nanosaur_ros2_control/>
+        <xacro:nanosaur_ros2_control robot_name="$(arg robot_name)" />
     </xacro:if>
     <!-- nanosaur differential drive controller -->

Commit message: First rearrange nanosaur ignition package

File: nanosaur_ignition/urdf/nanosaur.ignition.xacro (robot description, xacro)
@@ -11,6 +11,7 @@
     <xacro:arg name="robot_name" default="nanosaur" />
     <!-- camera definitions -->
-    <xacro:arg name="cover_type" default="fisheye" /> <!--options pi, fisheye, realsense, zedmini -->
-    <xacro:property name="cover_type_name" value="$(arg cover_type)" />
+    <xacro:arg name="head_type" default="empty" /> <!--options: empty, realsense, zedmini -->
+    <xacro:arg name="flap_type" default="empty" /> <!--options: empty, LD06 -->
+    <xacro:property name="cover_type_name" value="$(arg head_type)" />
     <!-- control definitions -->
     <xacro:property name="control_type_name" value="ros2_control" /> <!--options ros2_control, diff_drive -->
@@ -23,5 +24,12 @@
          Add extra wheel and center sprocket for differential drive simulation -->
     <!--https://github.com/ros-simulation/gazebo_ros_pkgs/pull/1284 -->
-    <xacro:nanosaur cover_type="$(arg cover_type)"
+    <link name="base_link" />
+    <joint name="nanosaur_base_joint" type="fixed">
+        <origin xyz="0 0 0.05" rpy="0 0 0" />
+        <parent link="base_link"/>
+        <child link="nanosaur_base"/>
+    </joint>
+    <xacro:nanosaur head_type="$(arg head_type)"
+                    flap_type="$(arg flap_type)"
                     use_nominal_extrinsics="true"
                     diff_drive_emulation="true"/>
@@ -39,15 +47,6 @@
     </xacro:if>
     <!-- Nanosaur sensors -->
-    <xacro:if value="${cover_type_name == 'pi'}">
-        <xacro:normal_camera parent_name="camera_board" sensor_name="camera" robot_name="$(arg robot_name)">
-            <origin xyz="0 0 0" rpy="0 -${M_PI/2} 0" />
-        </xacro:normal_camera>
-    </xacro:if>
-    <xacro:if value="${cover_type_name == 'fisheye'}">
-    </xacro:if>
     <xacro:if value="${cover_type_name == 'realsense'}">
         <xacro:realsense_camera parent_name="camera_board" sensor_name="camera" robot_name="$(arg robot_name)" publish_pointcloud="$(arg publish_pointcloud)" />
     </xacro:if>
-    <xacro:if value="${cover_type_name == 'zed'}">
-    </xacro:if>
 </robot>

Commit message: Improve nanosaur simulation

File: nanosaur_ignition/urdf/nanosaur.ignition.xacro (robot description, xacro)
@@ -4,8 +4,6 @@
     <xacro:include filename="$(find nanosaur_description)/urdf/robot.urdf.xacro" />
     <!-- differential drive -->
-    <xacro:include filename="$(find nanosaur_ignition)/urdf/diff_drive.ignition.xacro" />
-    <xacro:include filename="$(find nanosaur_ignition)/urdf/ros2_control.ignition.xacro" />
+    <xacro:include filename="$(find nanosaur_ignition)/urdf/mecanum.ignition.xacro" />
     <!-- Sensors -->
-    <xacro:include filename="$(find nanosaur_ignition)/urdf/sensors/camera.ignition.xacro" />
     <xacro:include filename="$(find nanosaur_ignition)/urdf/sensors/realsense.ignition.xacro" />
     <xacro:arg name="robot_name" default="nanosaur" />
@@ -14,6 +12,4 @@
     <xacro:arg name="flap_type" default="empty" /> <!--options: empty, LD06 -->
     <xacro:property name="cover_type_name" value="$(arg head_type)" />
-    <!-- control definitions -->
-    <xacro:property name="control_type_name" value="ros2_control" /> <!--options ros2_control, diff_drive -->
     <xacro:arg name="publish_pointcloud"  default="false"/>
     <xacro:arg name="publish_odom_tf"  default="false"/>
@@ -21,6 +17,6 @@
     <xacro:arg name="resolution"    default="VGA"/>
     <!-- nanosaur robot
-         "diff_drive_emulation" parameter enable simulation mode.
-         Add extra wheel and center sprocket for differential drive simulation -->
+        "diff_drive_emulation" parameter enable simulation mode.
+        Add extra wheel and center sprocket for differential drive simulation -->
     <!--https://github.com/ros-simulation/gazebo_ros_pkgs/pull/1284 -->
     <link name="base_link" />
@@ -34,16 +30,6 @@
                     use_nominal_extrinsics="true"
                     diff_drive_emulation="true"/>
-    <xacro:if value="${control_type_name == 'ros2_control'}">
-        <xacro:nanosaur_ros2_control robot_name="$(arg robot_name)" />
-    </xacro:if>
-    <!-- nanosaur differential drive controller -->
-    <xacro:if value="${control_type_name == 'diff_drive'}">
-        <xacro:track_drive parent="base_link"
-                        robot_name="$(arg robot_name)"
-                        update_rate="100.0"
-                        wheel_radius="0.0150"
-                        wheel_separation="0.4"
-                        publish_odom_tf="$(arg publish_odom_tf)" />
-    </xacro:if>
+    <!-- nanosaur mecanum wheel drive controller -->
+    <xacro:mecanum_drive parent="base_link" wheelbase="0.1" wheel_radius="0.0185" wheel_separation="0.082" />
     <!-- Nanosaur sensors -->
     <xacro:if value="${cover_type_name == 'realsense'}">
